File: baseline/baseline.kicad_pcb (KiCad board)
At the start: 2 copper layers, 18 parts, among them J1 TYPE-C-31-M-12, SW1 TS-1088-AR02016, SW2 TS-1088-AR02016, U3 LD1117S33TR_SOT223

Commit message: ESP dev-board generator: on-board LED wiring + GPIO-safety curation + routing robustness
Wire the skeleton's BUILTIN_LED net to a safe module GPIO on every board.
board.yaml gains structured strapping/input_only lists + a builtin_led pin; the
generator picks the safe (I/O-capable, non-strapping, broken-out) pad physically
NEAREST the on-board LED on the laid-out PCB (shortest trace) and aliases
BUILTIN_LED onto that pin's GPIOxx net. build_board hard-errors if builtin_led is
a strapping / input-only / non-broken-out pin. All 12 boards now wire the LED and
route fully connected + DRC-clean.

- build_board.py: resolve_led_pin (build-time safety gate) + pick_builtin_led
  (nearest-pad heuristic), BUILTIN_LED alias on a wire stub, PCB pad-net override,
  breakout_split helper.
- place_pcb.py: extract compute_layout() + add net_pad_global() so the picker can
  reuse the real placement geometry.
- route_board.py: remove the <M>.routing.* temp project companions KiCad spawns,
  so routing is genuinely in place (only <M>.kicad_pcb changes).
- route_all.py: strict gate — fail on any non-GND real DRC. CC-vs-NPTH is fixed by
  the USB-C NPTH 0.3mm pad clearance (>= the 0.254mm DRU rule), no longer accepted.
- board.yaml x12: strapping/input_only/builtin_led curated from atomic14 data.
- baseline: BUILTIN_LED LED net + USB-C NPTH clearance/DRU fixes enabling the above.
- docs (README/DECISIONS/AGENT_END_TO_END): new board.yaml schema + heuristics.

Co-Authored-By: Claude Opus 4.8 (1M context) <noreply@anthropic.com>
Parts:
- moved R3 1.78 mm to (153.4, 75.2)
- moved C5 1.75 mm to (153.4, 77.0)
- turned C1 to 180 degrees
- turned C2 to 180 degrees
- turned C3 to 180 degrees
- turned C4 to 90 degrees
- turned R4 to 0 degrees
- turned R5 to 0 degrees
Connections:
- net GPIO21 renamed BUILTIN_LED
Changed lines of the file:
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@@
 	(footprint "Resistor_SMD:R_0603_1608Metric"
 		(layer "F.Cu")
-		(at 153.353 76.962 180)
+		(at 153.416 75.184 180)
 		(descr "Resistor SMD 0603 (1608 Metric), square (rectangular) end terminal, IPC-7351 nominal, (Body size source: IPC-SM-782 page 72, https://www.pcb-3d.com/wordpress/wp-content/uploads/ipc-sm-782a_amendment_1_and_2.pdf)")
 		(tags "resistor")
@@
 	(footprint "Capacitor_SMD:C_0603_1608Metric"
 		(layer "F.Cu")
-		(at 164.592 73.927 -90)
+		(at 164.592 73.927 90)
 		(descr "Capacitor SMD 0603 (1608 Metric), square (rectangular) end terminal, IPC-7351 nominal, (Body size source: IPC-SM-782 page 76, https://www.pcb-3d.com/wordpress/wp-content/uploads/ipc-sm-782a_amendment_1_and_2.pdf)")
 		(tags "capacitor")
@@
 		(duplicate_pad_numbers_are_jumpers no)
 		(fp_line
-			(start -0.14058 0.51)
-			(end 0.14058 0.51)
+			(start -0.14058 -0.51)
+			(end 0.14058 -0.51)
 			(stroke
 				(width 0.12)
@@
 		)
 		(fp_line
-			(start -0.14058 -0.51)
-			(end 0.14058 -0.51)
+			(start -0.14058 0.51)
+			(end 0.14058 0.51)
 			(stroke
 				(width 0.12)
@@
 		)
 		(pad "1" smd roundrect
-			(at -0.775 0 270)
+			(at -0.775 0 90)
 			(size 0.9 0.95)
 			(layers "F.Cu" "F.Mask" "F.Paste")
@@
 		)
 		(pad "2" smd roundrect
-			(at 0.775 0 270)
+			(at 0.775 0 90)
 			(size 0.9 0.95)
 			(layers "F.Cu" "F.Mask" "F.Paste")
@@
 	(footprint "Capacitor_SMD:C_0603_1608Metric"
 		(layer "F.Cu")
-		(at 153.403 73.406)
+		(at 153.403 73.406 180)
 		(descr "Capacitor SMD 0603 (1608 Metric), square (rectangular) end terminal, IPC-7351 nominal, (Body size source: IPC-SM-782 page 76, https://www.pcb-3d.com/wordpress/wp-content/uploads/ipc-sm-782a_amendment_1_and_2.pdf)")
 		(tags "capacitor")
 		(property "Reference" "C3"
-			(at -2.527 0.06 0)
+			(at 2.527 0 0)
 			(layer "F.SilkS")
 			(effects
@@
 		(duplicate_pad_numbers_are_jumpers no)
 		(fp_line
-			(start -0.14058 -0.51)
-			(end 0.14058 -0.51)
+			(start -0.14058 0.51)
+			(end 0.14058 0.51)
 			(stroke
 				(width 0.12)
@@
 		)
 		(fp_line
-			(start -0.14058 0.51)
-			(end 0.14058 0.51)
+			(start -0.14058 -0.51)
+			(end 0.14058 -0.51)
 			(stroke
 				(width 0.12)
@@
 		)
 		(pad "1" smd roundrect
-			(at -0.775 0)
+			(at -0.775 0 180)
 			(size 0.9 0.95)
 			(layers "F.Cu" "F.Mask" "F.Paste")
@@
 		)
 		(pad "2" smd roundrect
-			(at 0.775 0)
+			(at 0.775 0 180)
 			(size 0.9 0.95)
 			(layers "F.Cu" "F.Mask" "F.Paste")
@@
 	(footprint "Capacitor_SMD:C_0603_1608Metric"
 		(layer "F.Cu")
-		(at 153.416 75.214)
+		(at 153.416 76.962)
 		(descr "Capacitor SMD 0603 (1608 Metric), square (rectangular) end terminal, IPC-7351 nominal, (Body size source: IPC-SM-782 page 76, https://www.pcb-3d.com/wordpress/wp-content/uploads/ipc-sm-782a_amendment_1_and_2.pdf)")
 		(tags "capacitor")
@@
 		(sheetname "/")
 		(sheetfile "baseline.kicad_sch")
+		(units
+			(unit
+				(name "A")
+				(pins "A5" "A6" "A7" "A8" "A4_B9" "B4_A9" "B8" "B7" "B6" "B5" "S1" "S2"
+					"S3" "S4" "A1_B12" "B1_A12"
+				)
+			)
+		)
 		(attr smd)
 		(duplicate_pad_numbers_are_jumpers no)
@@
 			(drill 0.6)
 			(layers "*.Cu" "*.Mask")
-			(clearance 0.2)
+			(clearance 0.3)
 		)
 		(pad "" np_thru_hole circle
@@
 			(drill 0.6)
 			(layers "*.Cu" "*.Mask")
-			(clearance 0.2)
+			(clearance 0.3)
 		)
 		(pad "A1_B12" smd rect
@@
 	(footprint "Capacitor_SMD:C_0603_1608Metric"
 		(layer "F.Cu")
-		(at 153.403 69.85)
+		(at 153.403 69.85 180)
 		(descr "Capacitor SMD 0603 (1608 Metric), square (rectangular) end terminal, IPC-7351 nominal, (Body size source: IPC-SM-782 page 76, https://www.pcb-3d.com/wordpress/wp-content/uploads/ipc-sm-782a_amendment_1_and_2.pdf)")
 		(tags "capacitor")
 		(property "Reference" "C1"
-			(at -2.527 0 0)
+			(at 2.527 0 0)
 			(layer "F.SilkS")
 			(effects
@@
 		(duplicate_pad_numbers_are_jumpers no)
 		(fp_line
-			(start -0.14058 -0.51)
-			(end 0.14058 -0.51)
+			(start -0.14058 0.51)
+			(end 0.14058 0.51)
 			(stroke
 				(width 0.12)
@@
 		)
 		(fp_line
-			(start -0.14058 0.51)
-			(end 0.14058 0.51)
+			(start -0.14058 -0.51)
+			(end 0.14058 -0.51)
 			(stroke
 				(width 0.12)
@@
 		)
 		(pad "1" smd roundrect
-			(at -0.775 0)
+			(at -0.775 0 180)
 			(size 0.9 0.95)
 			(layers "F.Cu" "F.Mask" "F.Paste")
@@
 		)
 		(pad "2" smd roundrect
-			(at 0.775 0)
+			(at 0.775 0 180)
 			(size 0.9 0.95)
 			(layers "F.Cu" "F.Mask" "F.Paste")
@@
 	(footprint "Resistor_SMD:R_0603_1608Metric"
 		(layer "F.Cu")
-		(at 167.3605 72.136 180)
+		(at 167.3605 72.136)
 		(descr "Resistor SMD 0603 (1608 Metric), square (rectangular) end terminal, IPC-7351 nominal, (Body size source: IPC-SM-782 page 72, https://www.pcb-3d.com/wordpress/wp-content/uploads/ipc-sm-782a_amendment_1_and_2.pdf)")
 		(tags "resistor")
 		(property "Reference" "R5"
-			(at -2.54 0 0)
+			(at 2.5655 0 0)
 			(layer "F.SilkS")
 			(effects
@@
 		(duplicate_pad_numbers_are_jumpers no)
 		(fp_line
-			(start -0.237258 0.5225)
-			(end 0.237258 0.5225)
+			(start -0.237258 -0.5225)
+			(end 0.237258 -0.5225)
 			(stroke
 				(width 0.12)
@@
 		)
 		(fp_line
-			(start -0.237258 -0.5225)
-			(end 0.237258 -0.5225)
+			(start -0.237258 0.5225)
+			(end 0.237258 0.5225)
 			(stroke
 				(width 0.12)
@@
 		)
 		(pad "1" smd roundrect
-			(at -0.825 0 180)
+			(at -0.825 0)
 			(size 0.8 0.95)
 			(layers "F.Cu" "F.Mask" "F.Paste")
@@
 		)
 		(pad "2" smd roundrect
-			(at 0.825 0 180)
+			(at 0.825 0)
 			(size 0.8 0.95)
 			(layers "F.Cu" "F.Mask" "F.Paste")
@@
 	(footprint "Resistor_SMD:R_0603_1608Metric"
 		(layer "F.Cu")
-		(at 167.2975 75.692 180)
+		(at 167.2975 75.692)
 		(descr "Resistor SMD 0603 (1608 Metric), square (rectangular) end terminal, IPC-7351 nominal, (Body size source: IPC-SM-782 page 72, https://www.pcb-3d.com/wordpress/wp-content/uploads/ipc-sm-782a_amendment_1_and_2.pdf)")
 		(tags "resistor")
 		(property "Reference" "R4"
-			(at -2.603 0 0)
+			(at 2.6285 0 0)
 			(layer "F.SilkS")
 			(effects
@@
 		(duplicate_pad_numbers_are_jumpers no)
 		(fp_line
-			(start -0.237258 0.5225)
-			(end 0.237258 0.5225)
+			(start -0.237258 -0.5225)
+			(end 0.237258 -0.5225)
 			(stroke
 				(width 0.12)
@@
 		)
 		(fp_line
-			(start -0.237258 -0.5225)
-			(end 0.237258 -0.5225)
+			(start -0.237258 0.5225)
+			(end 0.237258 0.5225)
 			(stroke
 				(width 0.12)
@@
 		)
 		(pad "1" smd roundrect
-			(at -0.825 0 180)
+			(at -0.825 0)
 			(size 0.8 0.95)
 			(layers "F.Cu" "F.Mask" "F.Paste")
@@
 		)
 		(pad "2" smd roundrect
-			(at 0.825 0 180)
+			(at 0.825 0)
 			(size 0.8 0.95)
 			(layers "F.Cu" "F.Mask" "F.Paste")
@@
 			(layers "F.Cu" "F.Mask" "F.Paste")
 			(roundrect_rratio 0.25)
-			(net "GPIO21")
+			(net "BUILTIN_LED")
 			(pintype "passive")
 		)
@@
 	(footprint "Capacitor_SMD:C_0603_1608Metric"
 		(layer "F.Cu")
-		(at 153.403 71.628)
+		(at 153.403 71.628 180)
 		(descr "Capacitor SMD 0603 (1608 Metric), square (rectangular) end terminal, IPC-7351 nominal, (Body size source: IPC-SM-782 page 76, https://www.pcb-3d.com/wordpress/wp-content/uploads/ipc-sm-782a_amendment_1_and_2.pdf)")
 		(tags "capacitor")
 		(property "Reference" "C2"
-			(at -2.527 0.03 0)
+			(at 2.527 0 0)
 			(layer "F.SilkS")
 			(effects
@@
 		(duplicate_pad_numbers_are_jumpers no)
 		(fp_line
-			(start -0.14058 -0.51)
-			(end 0.14058 -0.51)
+			(start -0.14058 0.51)
+			(end 0.14058 0.51)
 			(stroke
 				(width 0.12)
@@
 		)
 		(fp_line
-			(start -0.14058 0.51)
-			(end 0.14058 0.51)
+			(start -0.14058 -0.51)
+			(end 0.14058 -0.51)
 			(stroke
 				(width 0.12)
@@
 		)
 		(pad "1" smd roundrect
-			(at -0.775 0)
+			(at -0.775 0 180)
 			(size 0.9 0.95)
 			(layers "F.Cu" "F.Mask" "F.Paste")
@@
 		)
 		(pad "2" smd roundrect
-			(at 0.775 0)
+			(at 0.775 0 180)
 			(size 0.9 0.95)
 			(layers "F.Cu" "F.Mask" "F.Paste")

Commit message: Routing pipeline: per-module BOOT mapping, by-side header allocation, GND-plane + via fixes
Build/schematic:
- BOOT net mapped to each module's actual boot/strapping GPIO (board.yaml `boot:`),
  mirroring the builtin_led alias — was hard-wired to GPIO0, wrong on RISC-V parts.
- breakout_split now allocates header pins BY PHYSICAL SIDE (left edge->left header,
  right edge->right, bottom by x) instead of a count midpoint, which dumped
  right-edge pins into the left header on unbalanced left/right-only modules
  (C5/C6-WROOM) so they routed across the board. Shorter header padded with GND.
- Deterministic UUIDs (uuid5 over a counter) so rebuilds are byte-identical;
  random uuid4s reshuffled route.py's net order and flipped marginal nets.

Routing (route_board):
- Fill the GND zone before routing so route.py sees the poured copper.
- GND excluded from the route pass (it's the poured plane, not a signal) +
  route_diff --no-gnd-vias: stop redundant GND vias crowding the diff pair.
- Differential-pair routing (--diff) is now the default; pre-routed baseline nets
  are skipped so hand-routed traces survive the autoroute.
- NPTH keepout rings (hole_keepouts.py) + --no-fix-drc-settings (issue #160) so the
  router respects our baseline DRC rules; via size 0.6->0.5mm.
- Single attempt then stop; per-stage debug snapshots under route_debug/.

Baseline: drop the 0.2mm USB-C footprint pad clearance overrides, BOOT net rename.

Co-Authored-By: Claude Opus 4.8 (1M context) <noreply@anthropic.com>
Connections:
- net GPIO0 renamed BOOT
Routing:
- net GND: track 0.00 -> 20.7 mm, vias 0 -> 7
- net +5V: track 0.00 -> 16.2 mm, vias 0 -> 2
- net EN: track 0.00 -> 6.85 mm
- net Net-(J1-CC1): track 0.00 -> 6.46 mm
- net Net-(J1-CC2): track 0.00 -> 6.17 mm
- net +3V3: track 0.00 -> 5.58 mm
- net D-: track 0.00 -> 2.54 mm
- net D+: track 0.00 -> 2.48 mm
- net Net-(D2-A): track 0.00 -> 2.45 mm
- net Net-(D1-A): track 0.00 -> 2.42 mm
- net Net-(D3-A): track 0.00 -> 1.79 mm
