File: baseline/baseline.kicad_sch (KiCad schematic)
At the start: 18 parts, among them J1 TYPE-C-31-M-12, SW1 TS-1088-AR02016, SW2 TS-1088-AR02016, U3 LD1117S33TR_SOT223

Commit message: ESP dev-board generator: on-board LED wiring + GPIO-safety curation + routing robustness
Wire the skeleton's BUILTIN_LED net to a safe module GPIO on every board.
board.yaml gains structured strapping/input_only lists + a builtin_led pin; the
generator picks the safe (I/O-capable, non-strapping, broken-out) pad physically
NEAREST the on-board LED on the laid-out PCB (shortest trace) and aliases
BUILTIN_LED onto that pin's GPIOxx net. build_board hard-errors if builtin_led is
a strapping / input-only / non-broken-out pin. All 12 boards now wire the LED and
route fully connected + DRC-clean.

- build_board.py: resolve_led_pin (build-time safety gate) + pick_builtin_led
  (nearest-pad heuristic), BUILTIN_LED alias on a wire stub, PCB pad-net override,
  breakout_split helper.
- place_pcb.py: extract compute_layout() + add net_pad_global() so the picker can
  reuse the real placement geometry.
- route_board.py: remove the <M>.routing.* temp project companions KiCad spawns,
  so routing is genuinely in place (only <M>.kicad_pcb changes).
- route_all.py: strict gate — fail on any non-GND real DRC. CC-vs-NPTH is fixed by
  the USB-C NPTH 0.3mm pad clearance (>= the 0.254mm DRU rule), no longer accepted.
- board.yaml x12: strapping/input_only/builtin_led curated from atomic14 data.
- baseline: BUILTIN_LED LED net + USB-C NPTH clearance/DRU fixes enabling the above.
- docs (README/DECISIONS/AGENT_END_TO_END): new board.yaml schema + heuristics.

Co-Authored-By: Claude Opus 4.8 (1M context) <noreply@anthropic.com>
Connections:
- net GPIO21 renamed BUILTIN_LED
Changed lines of the file:
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@@
 		)
 	)
-	(global_label "GPIO21"
+	(global_label "BUILTIN_LED"
 		(shape input)
 		(at 44.45 85.725 90)
@@
 		)
 		(property "Intersheetrefs" "${INTERSHEET_REFS}"
-			(at 44.45 75.8455 90)
+			(at 44.45 71.1888 90)
 			(hide yes)
 			(show_name no)

Commit message: Routing pipeline: per-module BOOT mapping, by-side header allocation, GND-plane + via fixes
Build/schematic:
- BOOT net mapped to each module's actual boot/strapping GPIO (board.yaml `boot:`),
  mirroring the builtin_led alias — was hard-wired to GPIO0, wrong on RISC-V parts.
- breakout_split now allocates header pins BY PHYSICAL SIDE (left edge->left header,
  right edge->right, bottom by x) instead of a count midpoint, which dumped
  right-edge pins into the left header on unbalanced left/right-only modules
  (C5/C6-WROOM) so they routed across the board. Shorter header padded with GND.
- Deterministic UUIDs (uuid5 over a counter) so rebuilds are byte-identical;
  random uuid4s reshuffled route.py's net order and flipped marginal nets.

Routing (route_board):
- Fill the GND zone before routing so route.py sees the poured copper.
- GND excluded from the route pass (it's the poured plane, not a signal) +
  route_diff --no-gnd-vias: stop redundant GND vias crowding the diff pair.
- Differential-pair routing (--diff) is now the default; pre-routed baseline nets
  are skipped so hand-routed traces survive the autoroute.
- NPTH keepout rings (hole_keepouts.py) + --no-fix-drc-settings (issue #160) so the
  router respects our baseline DRC rules; via size 0.6->0.5mm.
- Single attempt then stop; per-stage debug snapshots under route_debug/.

Baseline: drop the 0.2mm USB-C footprint pad clearance overrides, BOOT net rename.

Co-Authored-By: Claude Opus 4.8 (1M context) <noreply@anthropic.com>
Connections:
- net GPIO0 renamed BOOT
Other:
- moved on the sheet: J1
Changed lines of the file:
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@@
+	)
+	(junction
+		(at 74.93 30.48)
+		(diameter 0)
+		(color 0 0 0 0)
 	)
 	(junction
@@
 	)
 	(junction
+		(at 73.66 27.94)
+		(diameter 0)
+		(color 0 0 0 0)
+	)
+	(junction
 		(at 46.99 129.54)
 		(diameter 0)
@@
 	)
 	(no_connect
-		(at 70.485 25.4)
+		(at 68.58 25.4)
 	)
 	(no_connect
-		(at 34.925 33.02)
+		(at 33.02 33.02)
 	)
 	(wire
@@
 	(wire
 		(pts
-			(xy 70.485 38.1) (xy 70.485 40.64)
+			(xy 74.93 44.45) (xy 74.93 30.48)
+		)
+		(stroke
+			(width 0)
+			(type default)
+		)
+	)
+	(wire
+		(pts
+			(xy 30.48 30.48) (xy 30.48 43.18)
+		)
+		(stroke
+			(width 0)
+			(type default)
+		)
+	)
+	(wire
+		(pts
+			(xy 68.58 38.1) (xy 68.58 39.37)
 		)
 		(stroke
@@
 	(wire
 		(pts
+			(xy 30.48 43.18) (xy 73.66 43.18)
+		)
+		(stroke
+			(width 0)
+			(type default)
+		)
+	)
+	(wire
+		(pts
 			(xy 46.355 178.435) (xy 46.355 179.705)
 		)
@@
 	(wire
 		(pts
+			(xy 68.58 39.37) (xy 70.485 39.37)
+		)
+		(stroke
+			(width 0)
+			(type default)
+		)
+	)
+	(wire
+		(pts
 			(xy 70.485 63.5) (xy 86.36 63.5)
 		)
@@
 	(wire
 		(pts
+			(xy 74.93 30.48) (xy 68.58 30.48)
+		)
+		(stroke
+			(width 0)
+			(type default)
+		)
+	)
+	(wire
+		(pts
 			(xy 20.32 25.4) (xy 20.32 45.72)
 		)
@@
 	(wire
 		(pts
+			(xy 33.02 27.94) (xy 29.21 27.94)
+		)
+		(stroke
+			(width 0)
+			(type default)
+		)
+	)
+	(wire
+		(pts
 			(xy 46.355 179.705) (xy 46.355 180.975)
 		)
@@
 	(wire
 		(pts
+			(xy 29.21 27.94) (xy 29.21 44.45)
+		)
+		(stroke
+			(width 0)
+			(type default)
+		)
+	)
+	(wire
+		(pts
 			(xy 25.4 180.34) (xy 25.4 179.07)
 		)
@@
 	(wire
 		(pts
-			(xy 70.485 20.32) (xy 74.295 20.32)
+			(xy 68.58 20.32) (xy 74.295 20.32)
+		)
+		(stroke
+			(width 0)
+			(type default)
+		)
+	)
+	(wire
+		(pts
+			(xy 73.66 27.94) (xy 68.58 27.94)
 		)
 		(stroke
@@
 	(wire
 		(pts
-			(xy 20.32 25.4) (xy 34.925 25.4)
+			(xy 20.32 25.4) (xy 33.02 25.4)
+		)
+		(stroke
+			(width 0)
+			(type default)
+		)
+	)
+	(wire
+		(pts
+			(xy 68.58 40.64) (xy 70.485 40.64)
+		)
+		(stroke
+			(width 0)
+			(type default)
+		)
+	)
+	(wire
+		(pts
+			(xy 29.21 44.45) (xy 74.93 44.45)
+		)
+		(stroke
+			(width 0)
+			(type default)
+		)
+	)
+	(wire
+		(pts
+			(xy 70.485 39.37) (xy 70.485 40.64)
+		)
+		(stroke
+			(width 0)
+			(type default)
+		)
+	)
+	(wire
+		(pts
+			(xy 73.66 43.18) (xy 73.66 27.94)
 		)
 		(stroke
@@
 	(wire
 		(pts
+			(xy 33.02 30.48) (xy 30.48 30.48)
+		)
+		(stroke
+			(width 0)
+			(type default)
+		)
+	)
+	(wire
+		(pts
 			(xy 53.34 137.16) (xy 59.055 137.16)
 		)
@@
 	(wire
 		(pts
+			(xy 76.2 27.94) (xy 73.66 27.94)
+		)
+		(stroke
+			(width 0)
+			(type default)
+		)
+	)
+	(wire
+		(pts
 			(xy 44.45 100.965) (xy 44.45 106.68)
 		)
@@
 	(wire
 		(pts
-			(xy 70.485 33.02) (xy 86.36 33.02)
+			(xy 68.58 33.02) (xy 86.36 33.02)
+		)
+		(stroke
+			(width 0)
+			(type default)
+		)
+	)
+	(wire
+		(pts
+			(xy 76.2 30.48) (xy 74.93 30.48)
 		)
 		(stroke
@@
 	(global_label "D+"
 		(shape input)
-		(at 70.485 30.48 0)
+		(at 76.2 30.48 0)
 		(fields_autoplaced yes)
 		(effects
@@
 		)
 		(property "Intersheetrefs" "${INTERSHEET_REFS}"
-			(at 76.3126 30.48 0)
-			(hide yes)
-			(show_name no)
-			(do_not_autoplace no)
-			(effects
-				(font
-					(size 1.27 1.27)
-				)
-				(justify left)
-			)
-		)
-	)
-	(global_label "D-"
-		(shape input)
-		(at 34.925 30.48 180)
-		(fields_autoplaced yes)
-		(effects
-			(font
-				(size 1.27 1.27)
-			)
-			(justify right)
-		)
-		(property "Intersheetrefs" "${INTERSHEET_REFS}"
-			(at 29.0974 30.48 0)
-			(hide yes)
-			(show_name no)
-			(do_not_autoplace no)
-			(effects
-				(font
-					(size 1.27 1.27)
-				)
-				(justify right)
+			(at 82.0276 30.48 0)
+			(hide yes)
+			(show_name no)
+			(do_not_autoplace no)
+			(effects
+				(font
+					(size 1.27 1.27)
+				)
+				(justify left)
 			)
 		)
@@
 		)
 	)
-	(global_label "GPIO0"
+	(global_label "BOOT"
 		(shape input)
 		(at 25.4 163.83 90)
@@
 		)
 		(property "Intersheetrefs" "${INTERSHEET_REFS}"
-			(at 25.4 155.16 90)
+			(at 25.4 155.9462 90)
 			(hide yes)
 			(show_name no)
@@
 	(global_label "D-"
 		(shape input)
-		(at 70.485 27.94 0)
+		(at 76.2 27.94 0)
 		(fields_autoplaced yes)
 		(effects
@@
 		)
 		(property "Intersheetrefs" "${INTERSHEET_REFS}"
-			(at 76.3126 27.94 0)
-			(hide yes)
-			(show_name no)
-			(do_not_autoplace no)
-			(effects
-				(font
-					(size 1.27 1.27)
-				)
-				(justify left)
-			)
-		)
-	)
-	(global_label "D+"
-		(shape input)
-		(at 34.925 27.94 180)
-		(fields_autoplaced yes)
-		(effects
-			(font
-				(size 1.27 1.27)
-			)
-			(justify right)
-		)
-		(property "Intersheetrefs" "${INTERSHEET_REFS}"
-			(at 29.0974 27.94 0)
-			(hide yes)
-			(show_name no)
-			(do_not_autoplace no)
-			(effects
-				(font
-					(size 1.27 1.27)
-				)
-				(justify right)
+			(at 82.0276 27.94 0)
+			(hide yes)
+			(show_name no)
+			(do_not_autoplace no)
+			(effects
+				(font
+					(size 1.27 1.27)
+				)
+				(justify left)
 			)
 		)
@@
 	(symbol
 		(lib_id "TYPE-C-31-M-12:TYPE-C-31-M-12")
-		(at 52.705 30.48 0)
+		(at 50.8 30.48 0)
 		(unit 1)
 		(body_style 1)
@@
 		(fields_autoplaced yes)
 		(property "Reference" "J1"
-			(at 52.705 12.7 0)
+			(at 50.8 12.7 0)
 			(show_name no)
 			(do_not_autoplace no)
@@
 		)
 		(property "Value" "TYPE-C-31-M-12"
-			(at 52.705 15.24 0)
+			(at 50.8 15.24 0)
 			(show_name no)
 			(do_not_autoplace no)
@@
 		)
 		(property "Footprint" "BasicEsp32Footprints:HRO_TYPE-C-31-M-12"
-			(at 52.705 30.48 0)
+			(at 50.8 30.48 0)
 			(hide yes)
 			(show_name no)
@@
 		)
 		(property "Datasheet" ""
-			(at 52.705 30.48 0)
+			(at 50.8 30.48 0)
 			(hide yes)
 			(show_name no)
@@
 		)
 		(property "Description" ""
-			(at 52.705 30.48 0)
+			(at 50.8 30.48 0)
 			(hide yes)
 			(show_name no)
@@
 		)
 		(property "PARTREV" "2020.12.08"
-			(at 52.705 30.48 0)
+			(at 50.8 30.48 0)
 			(hide yes)
 			(show_name no)
@@
 		)
 		(property "MANUFACTURER" "HRO Electronics Co., Ltd."
-			(at 52.705 30.48 0)
+			(at 50.8 30.48 0)
 			(hide yes)
 			(show_name no)
@@
 		)
 		(property "SNAPEDA_PN" "TYPE-C-31-M-12"
-			(at 52.705 30.48 0)
+			(at 50.8 30.48 0)
 			(hide yes)
 			(show_name no)
@@
 		)
 		(property "MAXIMUM_PACKAGE_HEIGHT" "3.26 mm"
-			(at 52.705 30.48 0)
+			(at 50.8 30.48 0)
 			(hide yes)
 			(show_name no)
@@
 		)
 		(property "STANDARD" "Manufacturer Recommendations"
-			(at 52.705 30.48 0)
+			(at 50.8 30.48 0)
 			(hide yes)
 			(show_name no)
@@
 		)
 		(property "MF" "韩国韩荣"
-			(at 52.705 30.48 0)
+			(at 50.8 30.48 0)
 			(hide yes)
 			(show_name no)
@@
 		)
 		(property "MP" "TYPE-C-31-M-12"
-			(at 52.705 30.48 0)
-			(hide yes)
-			(show_name no)
+			(at 50.8 30.48 0)
+			(hide yes)
+			(show_name no)
