File: baseline-right-en/baseline.kicad_pcb (KiCad board)
At the start: 2 copper layers, 18 parts, among them J1 TYPE-C-31-M-12, SW1 TS-1088-AR02016, SW2 TS-1088-AR02016, U3 LD1117S33TR_SOT223

Commit message: 0.4mm power nets
Parts:
- turned C1 to 0 degrees
- turned C2 to 0 degrees
- turned C3 to 0 degrees
- turned R3 to 0 degrees
Routing:
- net +3V3: track 5.74 -> 11.9 mm
- net +5V: track 16.6 -> 10.9 mm
- net EN: track 7.35 -> 7.99 mm
Changed lines of the file:
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@@
 		(capping no)
 		(filling no)
+		(zone_defaults)
 		(pcbplotparams
 			(layerselection 0x00000000_00000000_55555555_5755f5ff)
@@
 	(footprint "Capacitor_SMD:C_0603_1608Metric"
 		(layer "F.Cu")
-		(at 166.344 73.66 180)
+		(at 166.344 73.66)
 		(descr "Capacitor SMD 0603 (1608 Metric), square (rectangular) end terminal, IPC-7351 nominal, (Body size source: IPC-SM-782 page 76, https://www.pcb-3d.com/wordpress/wp-content/uploads/ipc-sm-782a_amendment_1_and_2.pdf)")
 		(tags "capacitor")
@@
 		(duplicate_pad_numbers_are_jumpers no)
 		(fp_line
-			(start -0.14058 0.51)
-			(end 0.14058 0.51)
+			(start -0.14058 -0.51)
+			(end 0.14058 -0.51)
 			(stroke
 				(width 0.12)
@@
 		)
 		(fp_line
-			(start -0.14058 -0.51)
-			(end 0.14058 -0.51)
+			(start -0.14058 0.51)
+			(end 0.14058 0.51)
 			(stroke
 				(width 0.12)
@@
 		)
 		(pad "1" smd roundrect
-			(at -0.775 0 180)
+			(at -0.775 0)
 			(size 0.9 0.95)
 			(layers "F.Cu" "F.Mask" "F.Paste")
@@
 		)
 		(pad "2" smd roundrect
-			(at 0.775 0 180)
+			(at 0.775 0)
 			(size 0.9 0.95)
 			(layers "F.Cu" "F.Mask" "F.Paste")
@@
 	(footprint "Capacitor_SMD:C_0603_1608Metric"
 		(layer "F.Cu")
-		(at 166.344 71.882 180)
+		(at 166.344 71.882)
 		(descr "Capacitor SMD 0603 (1608 Metric), square (rectangular) end terminal, IPC-7351 nominal, (Body size source: IPC-SM-782 page 76, https://www.pcb-3d.com/wordpress/wp-content/uploads/ipc-sm-782a_amendment_1_and_2.pdf)")
 		(tags "capacitor")
@@
 		(duplicate_pad_numbers_are_jumpers no)
 		(fp_line
-			(start -0.14058 0.51)
-			(end 0.14058 0.51)
+			(start -0.14058 -0.51)
+			(end 0.14058 -0.51)
 			(stroke
 				(width 0.12)
@@
 		)
 		(fp_line
-			(start -0.14058 -0.51)
-			(end 0.14058 -0.51)
+			(start -0.14058 0.51)
+			(end 0.14058 0.51)
 			(stroke
 				(width 0.12)
@@
 		)
 		(pad "1" smd roundrect
-			(at -0.775 0 180)
+			(at -0.775 0)
 			(size 0.9 0.95)
 			(layers "F.Cu" "F.Mask" "F.Paste")
@@
 		)
 		(pad "2" smd roundrect
-			(at 0.775 0 180)
+			(at 0.775 0)
 			(size 0.9 0.95)
 			(layers "F.Cu" "F.Mask" "F.Paste")
@@
 	(footprint "Resistor_SMD:R_0603_1608Metric"
 		(layer "F.Cu")
-		(at 166.357 75.438 180)
+		(at 166.357 75.438)
 		(descr "Resistor SMD 0603 (1608 Metric), square (rectangular) end terminal, IPC-7351 nominal, (Body size source: IPC-SM-782 page 72, https://www.pcb-3d.com/wordpress/wp-content/uploads/ipc-sm-782a_amendment_1_and_2.pdf)")
 		(tags "resistor")
@@
 		(duplicate_pad_numbers_are_jumpers no)
 		(fp_line
-			(start -0.237258 0.5225)
-			(end 0.237258 0.5225)
+			(start -0.237258 -0.5225)
+			(end 0.237258 -0.5225)
 			(stroke
 				(width 0.12)
@@
 		)
 		(fp_line
-			(start -0.237258 -0.5225)
-			(end 0.237258 -0.5225)
+			(start -0.237258 0.5225)
+			(end 0.237258 0.5225)
 			(stroke
 				(width 0.12)
@@
 		)
 		(pad "1" smd roundrect
-			(at -0.825 0 180)
+			(at -0.825 0)
 			(size 0.8 0.95)
 			(layers "F.Cu" "F.Mask" "F.Paste")
@@
 		)
 		(pad "2" smd roundrect
-			(at 0.825 0 180)
+			(at 0.825 0)
 			(size 0.8 0.95)
 			(layers "F.Cu" "F.Mask" "F.Paste")
@@
 	(footprint "Capacitor_SMD:C_0603_1608Metric"
 		(layer "F.Cu")
-		(at 166.344 70.104 180)
+		(at 166.344 70.104)
 		(descr "Capacitor SMD 0603 (1608 Metric), square (rectangular) end terminal, IPC-7351 nominal, (Body size source: IPC-SM-782 page 76, https://www.pcb-3d.com/wordpress/wp-content/uploads/ipc-sm-782a_amendment_1_and_2.pdf)")
 		(tags "capacitor")
@@
 		(duplicate_pad_numbers_are_jumpers no)
 		(fp_line
-			(start -0.14058 0.51)
-			(end 0.14058 0.51)
+			(start -0.14058 -0.51)
+			(end 0.14058 -0.51)
 			(stroke
 				(width 0.12)
@@
 		)
 		(fp_line
-			(start -0.14058 -0.51)
-			(end 0.14058 -0.51)
+			(start -0.14058 0.51)
+			(end 0.14058 0.51)
 			(stroke
 				(width 0.12)
@@
 		)
 		(pad "1" smd roundrect
-			(at -0.775 0 180)
+			(at -0.775 0)
 			(size 0.9 0.95)
 			(layers "F.Cu" "F.Mask" "F.Paste")
@@
 		)
 		(pad "2" smd roundrect
-			(at 0.775 0 180)
+			(at 0.775 0)
 			(size 0.9 0.95)
 			(layers "F.Cu" "F.Mask" "F.Paste")
@@
 	)
 	(segment
-		(start 167.271 70.256)
-		(end 167.119 70.104)
-		(width 0.2)
-		(layer "F.Cu")
-		(net "+3V3")
-	)
-	(segment
-		(start 153.034 72.39)
-		(end 153.034 72.5555)
-		(width 0.15)
-		(layer "F.Cu")
-		(net "+3V3")
-	)
-	(segment
 		(start 167.182 75.438)
-		(end 167.182 70.167)
-		(width 0.2)
-		(layer "F.Cu")
-		(net "+3V3")
-	)
-	(segment
-		(start 167.182 70.167)
-		(end 167.119 70.104)
-		(width 0.2)
-		(layer "F.Cu")
-		(net "+3V3")
-	)
-	(segment
-		(start 165.582 75.488)
-		(end 165.532 75.438)
+		(end 167.182 75.616)
 		(width 0.15)
 		(layer "F.Cu")
@@
 	)
 	(segment
-		(start 165.582 77.216)
-		(end 165.582 75.488)
+		(start 167.182 75.616)
+		(end 165.582 77.216)
 		(width 0.15)
 		(layer "F.Cu")
@@
 	)
 	(segment
-		(start 157.734 79.756)
-		(end 154.94 76.962)
-		(width 0.2)
-		(layer "F.Cu")
-		(net "+5V")
-	)
-	(segment
-		(start 157.5955 79.8945)
-		(end 157.734 79.756)
-		(width 0.2)
-		(layer "F.Cu")
-		(net "+5V")
-	)
-	(segment
-		(start 162.3955 80.952)
-		(end 162.3955 79.756)
-		(width 0.2)
-		(layer "F.Cu")
-		(net "+5V")
-	)
-	(segment
-		(start 152.971 75.946)
-		(end 152.971 76.1745)
-		(width 0.15)
-		(layer "F.Cu")
-		(net "+5V")
-	)
-	(segment
-		(start 162.3955 79.756)
-		(end 162.3955 76.6315)
-		(width 0.2)
-		(layer "F.Cu")
-		(net "+5V")
-	)
-	(segment
-		(start 157.5955 80.952)
-		(end 157.5955 79.8945)
-		(width 0.2)
-		(layer "F.Cu")
-		(net "+5V")
-	)
-	(segment
-		(start 154.94 76.962)
-		(end 154.94 75.197)
-		(width 0.2)
-		(layer "F.Cu")
-		(net "+5V")
-	)
-	(segment
-		(start 162.3955 76.6315)
-		(end 162.066 76.302)
-		(width 0.2)
-		(layer "F.Cu")
-		(net "+5V")
-	)
-	(via
-		(at 162.3955 79.756)
-		(size 0.5)
-		(drill 0.3)
-		(layers "F.Cu" "B.Cu")
-		(net "+5V")
-	)
-	(via
-		(at 157.734 79.756)
-		(size 0.5)
-		(drill 0.3)
-		(layers "F.Cu" "B.Cu")
-		(net "+5V")
-	)
-	(segment
-		(start 157.734 79.756)
-		(end 162.3955 79.756)
-		(width 0.2)
-		(layer "B.Cu")
-		(net "+5V")
-	)
-	(segment
 		(start 156.7955 80.952)
 		(end 156.7955 80.0875)
@@
 	)
 	(segment
-		(start 165.569 68.86)
-		(end 165.595 68.834)
+		(start 167.271 70.256)
+		(end 167.119 70.104)
 		(width 0.2)
 		(layer "F.Cu")
@@
 	)
 	(segment
-		(start 165.569 73.66)
-		(end 165.569 68.86)
+		(start 167.119 73.66)
+		(end 167.119 69.355)
+		(width 0.4)
+		(layer "F.Cu")
+		(net "GND")
+	)
+	(segment
+		(start 167.182 70.167)
+		(end 167.119 70.104)
 		(width 0.2)
 		(layer "F.Cu")
@@
 	)
 	(segment
+		(start 167.119 69.355)
+		(end 167.386 69.088)
+		(width 0.4)
+		(layer "F.Cu")
+		(net "GND")
+	)
+	(segment
 		(start 154.419 74.168)
 		(end 154.94 73.647)
@@
 	)
 	(via
-		(at 165.595 68.834)
+		(at 152.9965 78.74)
 		(size 0.5)
 		(drill 0.3)
@@
 	)
 	(via
-		(at 152.9965 78.74)
+		(at 167.386 69.088)
 		(size 0.5)
 		(drill 0.3)
@@
 	)
 	(segment
+		(start 165.569 70.104)
+		(end 165.569 75.401)
+		(width 0.4)
+		(layer "F.Cu")
+		(net "+3V3")
+	)
+	(segment
+		(start 165.582 75.488)
+		(end 165.532 75.438)
+		(width 0.15)
+		(layer "F.Cu")
+		(net "+3V3")
+	)
+	(segment
+		(start 153.034 72.39)
+		(end 153.034 72.5555)
+		(width 0.15)
+		(layer "F.Cu")
+		(net "+3V3")
+	)
+	(segment
+		(start 165.569 75.401)
+		(end 165.532 75.438)
+		(width 0.4)
+		(layer "F.Cu")
+		(net "+3V3")
+	)
+	(segment
+		(start 159.766 76.302)
+		(end 159.766 70.002)
+		(width 0.4)
+		(layer "F.Cu")
+		(net "+3V3")
+	)
+	(segment
+		(start 162.3955 79.756)
+		(end 162.3955 76.6315)
+		(width 0.4)
+		(layer "F.Cu")
+		(net "+5V")
+	)
+	(segment
+		(start 157.5955 79.8715)
+		(end 157.48 79.756)
+		(width 0.4)
+		(layer "F.Cu")
+		(net "+5V")
+	)
+	(segment
+		(start 162.3955 76.6315)
+		(end 162.066 76.302)
+		(width 0.4)
+		(layer "F.Cu")
+		(net "+5V")
+	)
+	(segment
+		(start 162.3955 80.952)
+		(end 162.3955 79.756)
+		(width 0.4)
+		(layer "F.Cu")
+		(net "+5V")
+	)
+	(segment
+		(start 157.5955 80.952)
+		(end 157.5955 79.8715)
+		(width 0.4)
+		(layer "F.Cu")
+		(net "+5V")
+	)
+	(via
+		(at 162.3955 79.756)
+		(size 0.5)
+		(drill 0.3)
+		(layers "F.Cu" "B.Cu")
+		(net "+5V")
+	)
+	(via
+		(at 157.48 79.756)
+		(size 0.5)
+		(drill 0.3)
+		(layers "F.Cu" "B.Cu")
+		(net "+5V")
+	)
+	(segment
+		(start 157.48 79.756)
+		(end 162.3955 79.756)
+		(width 0.4)
+		(layer "B.Cu")
+		(net "+5V")
+	)
+	(segment
 		(start 151.321 77.6235)
 		(end 151.4215 77.724)
@@
 	)
 	(segment
+		(start 151.384 70.5745)
+		(end 151.4215 70.612)
+		(width 0.15)
+		(layer "F.Cu")
+		(net "Net-(D3-A)")
+	)
+	(segment
+		(start 151.384 68.834)
+		(end 151.384 70.5745)
+		(width 0.15)
+		(layer "F.Cu")
+		(net "Net-(D3-A)")
+	)
+	(segment
 		(start 153.924 83.883)
 		(end 156.5345 83.883)
@@
 		(net "Net-(J1-CC2)")
 	)
-	(segment
-		(start 151.384 70.5745)
-		(end 151.4215 70.612)
-		(width 0.15)
-		(layer "F.Cu")
-		(net "Net-(D3-A)")
-	)
-	(segment
-		(start 151.384 68.834)
-		(end 151.384 70.5745)
-		(width 0.15)
-		(layer "F.Cu")
-		(net "Net-(D3-A)")
-	)
 	(embedded_fonts no)
