File: baseline-left-en/baseline.kicad_pcb (KiCad board)
At the start: 2 copper layers, 18 parts, among them J1 TYPE-C-31-M-12, SW1 TS-1088-AR02016, SW2 TS-1088-AR02016, U3 LD1117S33TR_SOT223

Commit message: baseline: tweak BOOT/EN button footprint silkscreen + re-save boards
Co-Authored-By: Claude Opus 4.8 (1M context) <noreply@anthropic.com>
Changed lines of the file:
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@@
 		(capping no)
 		(filling no)
-		(zone_defaults)
 		(pcbplotparams
 			(layerselection 0x00000000_00000000_55555555_5755f5ff)
@@
 		(sheetname "/")
 		(sheetfile "baseline.kicad_sch")
-		(units
-			(unit
-				(name "A")
-				(pins "1" "2")
-			)
-		)
 		(attr smd)
 		(duplicate_pad_numbers_are_jumpers no)
@@
 		(fp_line
 			(start -2.03 -1.54)
-			(end -2.03 -0.88)
+			(end -2.03 -1.13)
 			(stroke
 				(width 0.15)
@@
 		(fp_line
 			(start -2.03 1.54)
-			(end -2.03 0.88)
+			(end -2.03 1.21)
 			(stroke
 				(width 0.15)
@@
 		(sheetname "/")
 		(sheetfile "baseline.kicad_sch")
-		(units
-			(unit
-				(name "A")
-				(pins "1" "2")
-			)
-		)
 		(attr smd)
 		(duplicate_pad_numbers_are_jumpers no)
@@
 		(fp_line
 			(start -2.03 -1.54)
-			(end -2.03 -0.88)
+			(end -2.03 -1.13)
 			(stroke
 				(width 0.15)
@@
 		(fp_line
 			(start -2.03 1.54)
-			(end -2.03 0.88)
+			(end -2.03 1.21)
 			(stroke
 				(width 0.15)
